Commit message: renamed URDF objects

File: assets/atom_full.urdf (robot description, URDF)
Before this commit: robot cengaver, 22 links, 21 joints
Links:
- removed link cengaver
- added link atom
Joints:
- removed joint cengaver_to_Body
- added joint atom_to_Body: type fixed, parent atom, child Body, origin xyz=0 0 0.355
