Commit message: fixed depth camera and lidar structure in URDF

File: assets/atom_full.urdf (robot description, URDF)
Before this commit: robot atom, 22 links, 21 joints
Links:
- added link atom_body
- added link camera_sensor
- added link depth_sensor
- added link gpu_lidar
Joints:
- removed joint atom_to_Body
- removed joint lidar_joint
- added joint LIDAR_Body: type fixed, parent Body, child Lidar_Link, origin xyz=-0.015 0 -0.115 rpy=0 0 0
- added joint Lidar_Link_gpu_lidar: type fixed, parent Lidar_Link, child gpu_lidar, origin xyz=0 0 0 rpy=0 0 0
- added joint atom_body_to_Body: type fixed, parent atom_body, child Body
- added joint atom_to_atom_body: type fixed, parent atom, child atom_body
- added joint depth_camera_camera_sensor: type fixed, parent depth_camera, child camera_sensor, origin xyz=0 0 0 rpy=0 0 0
- added joint depth_camera_depth_sensor: type fixed, parent depth_camera, child depth_sensor, origin xyz=0 0 0 rpy=0 0 0
